Commit message: 1

File: legged_gym/resources/robots/bhr8fc2/BHR8FC2.urdf (robot description, URDF)
Before this commit: robot BHR8FC2, 21 links, 20 joints
Links:
- removed link lankle
- removed link lbigarm
- removed link lcalf
- removed link lfoot
- removed link lforearm
- removed link lhip1
- removed link lhip2
- removed link lshoulder1
- removed link lshoulder2
- removed link lthigh
- removed link rankle
- removed link rbigarm
- removed link rcalf
- removed link rfoot
- removed link rforearm
- removed link rhip1
- removed link rhip2
- removed link rshoulder1
- removed link rshoulder2
- removed link rthigh
- removed link torso
- added link left_ankle_pitch_link, mass 0.168311; collision mesh filename=meshes/left_ankle_pitch_link.stl; visual mesh filename=meshes/left_ankle_pitch_link.stl
- added link left_ankle_roll_link, mass 1.581270; collision mesh filename=meshes/left_ankle_roll_link.stl; visual mesh filename=meshes/left_ankle_roll_link.stl
- added link left_elbow_link, mass 0.181283; collision mesh filename=meshes/left_elbow_link.stl; visual mesh filename=meshes/left_elbow_link.stl
- added link left_hip_pitch_link, mass 3.096463; collision mesh filename=meshes/left_hip_pitch_link.stl; visual mesh filename=meshes/left_hip_pitch_link.stl
- added link left_hip_roll_link, mass 2.507222; collision mesh filename=meshes/left_hip_roll_link.stl; visual mesh filename=meshes/left_hip_roll_link.stl
- added link left_hip_yaw_link, mass 2.389579; collision mesh filename=meshes/left_hip_yaw_link.stl; visual mesh filename=meshes/left_hip_yaw_link.stl
- added link left_knee_link, mass 1.914266; collision mesh filename=meshes/left_knee_link.stl; visual mesh filename=meshes/left_knee_link.stl
- added link left_shoulder_pitch_link, mass 1.938195; collision mesh filename=meshes/left_shoulder_pitch_link.stl; visual mesh filename=meshes/left_shoulder_pitch_link.stl
- added link left_shoulder_roll_link, mass 2.116461; collision mesh filename=meshes/left_shoulder_roll_link.stl; visual mesh filename=meshes/left_shoulder_roll_link.stl
- added link left_shoulder_yaw_link, mass 1.703058; collision mesh filename=meshes/left_shoulder_yaw_link.stl; visual mesh filename=meshes/left_shoulder_yaw_link.stl
- added link right_ankle_pitch_link, mass 0.168311; collision mesh filename=meshes/right_ankle_pitch_link.stl; visual mesh filename=meshes/right_ankle_pitch_link.stl
- added link right_ankle_roll_link, mass 1.581376; collision mesh filename=meshes/right_ankle_roll_link.stl; visual mesh filename=meshes/right_ankle_roll_link.stl
- added link right_elbow_link, mass 0.181283; collision mesh filename=meshes/right_elbow_link.stl; visual mesh filename=meshes/right_elbow_link.stl
- added link right_hip_pitch_link, mass 3.096463; collision mesh filename=meshes/right_hip_pitch_link.stl; visual mesh filename=meshes/right_hip_pitch_link.stl
- added link right_hip_roll_link, mass 2.507088; collision mesh filename=meshes/right_hip_roll_link.stl; visual mesh filename=meshes/right_hip_roll_link.stl
- added link right_hip_yaw_link, mass 2.389579; collision mesh filename=meshes/right_hip_yaw_link.stl; visual mesh filename=meshes/right_hip_yaw_link.stl
- added link right_knee_link, mass 1.914266; collision mesh filename=meshes/right_knee_link.stl; visual mesh filename=meshes/right_knee_link.stl
- added link right_shoulder_pitch_link, mass 1.938195; collision mesh filename=meshes/right_shoulder_pitch_link.stl; visual mesh filename=meshes/right_shoulder_pitch_link.stl
- added link right_shoulder_roll_link, mass 2.116461; collision mesh filename=meshes/right_shoulder_roll_link.stl; visual mesh filename=meshes/right_shoulder_roll_link.stl
- added link right_shoulder_yaw_link, mass 1.703058; collision mesh filename=meshes/right_shoulder_yaw_link.stl; visual mesh filename=meshes/right_shoulder_yaw_link.stl
- added link torso_link, mass 22.905686; collision mesh filename=meshes/torso_link.stl; visual mesh filename=meshes/torso_link.stl
Joints:
- removed joint lankle1
- removed joint lankle2
- removed joint lelbow
- removed joint lhipPitch
- removed joint lhipRoll
- removed joint lhipYaw
- removed joint lknee
- removed joint lshoulderPitch
- removed joint lshoulderRoll
- removed joint lshoulderYaw
- removed joint rankle1
- removed joint rankle2
- removed joint relbow
- removed joint rhipPitch
- removed joint rhipRoll
- removed joint rhipYaw
- removed joint rknee
- removed joint rshoulderPitch
- removed joint rshoulderRoll
- removed joint rshoulderYaw
- added joint left_ankle_pitch_joint: type continuous, parent left_knee_link, child left_ankle_pitch_link, origin xyz=0 0 -0.35 rpy=0 0 0, axis 0 -1 0
- added joint left_ankle_roll_joint: type continuous, parent left_ankle_pitch_link, child left_ankle_roll_link, origin xyz=0.0410000000000001 0 0 rpy=0 0 0, axis -1 0 0
- added joint left_elbow_joint: type continuous, parent left_shoulder_yaw_link, child left_elbow_link, origin xyz=0 0.0099999999999949 -0.30324 rpy=0 0 0, axis 0 1 0
- added joint left_hip_pitch_joint: type continuous, parent left_hip_roll_link, child left_hip_pitch_link, origin xyz=0.0550000000000005 0.000100000001382744 0 rpy=0 0 0, axis 0 -1 0
- added joint left_hip_roll_joint: type continuous, parent left_hip_yaw_link, child left_hip_roll_link, origin xyz=-0.054 0 -0.13924 rpy=0 0 0, axis -1 0 0
- added joint left_hip_yaw_joint: type continuous, parent torso_link, child left_hip_yaw_link, origin xyz=0 0.0999999999999999 0.02324 rpy=0 0 0, axis 0 0 1
- added joint left_knee_joint: type continuous, parent left_hip_pitch_link, child left_knee_link, origin xyz=0 0 -0.375 rpy=0 0 0, axis 0 -1 0
- added joint left_shoulder_pitch_joint: type continuous, parent torso_link, child left_shoulder_pitch_link, origin xyz=-0.0262500000000013 0.13476 0.389 rpy=0 0 0, axis 0 1 0
- added joint left_shoulder_roll_joint: type continuous, parent left_shoulder_pitch_link, child left_shoulder_roll_link, origin xyz=-0.049 0.0842399999999999 0 rpy=0 0 0, axis 1 0 0
- added joint left_shoulder_yaw_joint: type continuous, parent left_shoulder_roll_link, child left_shoulder_yaw_link, origin xyz=0.049 0 -0.04976 rpy=0 0 0, axis 0 0 1
- added joint right_ankle_pitch_joint: type continuous, parent right_knee_link, child right_ankle_pitch_link, origin xyz=0 0 -0.349999999999999 rpy=0 0 0, axis 0 1 0
- added joint right_ankle_roll_joint: type continuous, parent right_ankle_pitch_link, child right_ankle_roll_link, origin xyz=0.0410000000000016 0 0 rpy=0 0 0, axis 1 0 0
- added joint right_elbow_joint: type continuous, parent right_shoulder_yaw_link, child right_elbow_link, origin xyz=0 -0.0100000000000002 -0.30324 rpy=0 0 0, axis 0 -1 0
- added joint right_hip_pitch_joint: type continuous, parent right_hip_roll_link, child right_hip_pitch_link, origin xyz=0.0550000000000002 -9.99999986171368E-05 0 rpy=0 0 0, axis 0 1 0
- added joint right_hip_roll_joint: type continuous, parent right_hip_yaw_link, child right_hip_roll_link, origin xyz=-0.054 0 -0.13924 rpy=0 0 0, axis -1 0 0
- added joint right_hip_yaw_joint: type continuous, parent torso_link, child right_hip_yaw_link, origin xyz=0 -0.1 0.02324 rpy=0 0 0, axis 0 0 1
- added joint right_knee_joint: type continuous, parent right_hip_pitch_link, child right_knee_link, origin xyz=0 0 -0.375 rpy=0 0 0, axis 0 1 0
- added joint right_shoulder_pitch_joint: type continuous, parent torso_link, child right_shoulder_pitch_link, origin xyz=-0.0262500000000002 -0.13476 0.389 rpy=0 0 0, axis 0 -1 0
- added joint right_shoulder_roll_joint: type continuous, parent right_shoulder_pitch_link, child right_shoulder_roll_link, origin xyz=-0.049 -0.0842399999999996 0 rpy=0 0 0, axis 1 0 0
- added joint right_shoulder_yaw_joint: type continuous, parent right_shoulder_roll_link, child right_shoulder_yaw_link, origin xyz=0.049 0 -0.0497599999999999 rpy=0 0 0, axis 0 0 1

Commit message: 1

File: legged_gym/resources/robots/bhr8fc2/BHR8FC2.urdf (robot description, URDF)
Before this commit: robot BHR8FC2, 21 links, 20 joints
Links:
- added link head_link, mass 0.618693; collision mesh filename=meshes/head_link.stl; visual mesh filename=meshes/head_link.stl
- link torso_link: mass 22.905686 -> 22.473048
Joints:
- added joint head_link_joint: type fixed, parent torso_link, child head_link, origin xyz=0.03 0 0.493594020755785 rpy=0 0 0, axis 0 0 0

Commit message: 1

File: legged_gym/resources/robots/bhr8fc2/BHR8FC2.urdf (robot description, URDF)
Before this commit: robot BHR8FC2, 22 links, 21 joints
Joints:
- removed joint head_link_joint
- added joint head_joint: type fixed, parent torso_link, child head_link, origin xyz=0.03 0 0.493594020755785 rpy=0 0 0, axis 0 0 0

Commit message: 1

File: legged_gym/resources/robots/bhr8fc2/BHR8FC2.urdf (robot description, URDF)
Before this commit: robot BHR8FC2, 22 links, 21 joints
Joints:
- joint left_ankle_pitch_joint: limit (none) -> lower=-0.87 upper=0.52 effort=40 velocity=30; type continuous -> revolute
- joint left_ankle_roll_joint: limit (none) -> lower=-0.35 upper=0.35 effort=40 velocity=30; type continuous -> revolute
- joint left_elbow_joint: limit (none) -> lower=0.0 upper=2.61 effort=100 velocity=30; type continuous -> revolute
- joint left_hip_pitch_joint: limit (none) -> lower=-1.92 upper=0.87 effort=200 velocity=30; type continuous -> revolute
- joint left_hip_roll_joint: limit (none) -> lower=-0.52 upper=0.52 effort=150 velocity=30; type continuous -> revolute
- joint left_hip_yaw_joint: limit (none) -> lower=-1.57 upper=1.57 effort=150 velocity=30; type continuous -> revolute
- joint left_knee_joint: limit (none) -> lower=0.0 upper=2.61 effort=200 velocity=30; type continuous -> revolute
- joint left_shoulder_pitch_joint: limit (none) -> lower=-2.87 upper=2.87 effort=100 velocity=30; type continuous -> revolute
- joint left_shoulder_roll_joint: limit (none) -> lower=-2.87 upper=2.87 effort=100 velocity=30; type continuous -> revolute
- joint left_shoulder_yaw_joint: limit (none) -> lower=-2.87 upper=2.87 effort=100 velocity=30; type continuous -> revolute
- joint right_ankle_pitch_joint: limit (none) -> lower=-0.87 upper=0.52 effort=40 velocity=30; type continuous -> revolute
- joint right_ankle_roll_joint: limit (none) -> lower=-0.35 upper=0.35 effort=40 velocity=30; type continuous -> revolute
- joint right_elbow_joint: limit (none) -> lower=0.0 upper=2.61 effort=100 velocity=30; type continuous -> revolute
- joint right_hip_pitch_joint: limit (none) -> lower=-1.92 upper=0.87 effort=200 velocity=30; type continuous -> revolute
- joint right_hip_roll_joint: limit (none) -> lower=-0.52 upper=0.52 effort=150 velocity=30; type continuous -> revolute
- joint right_hip_yaw_joint: limit (none) -> lower=-1.57 upper=1.57 effort=150 velocity=30; type continuous -> revolute
- joint right_knee_joint: limit (none) -> lower=0.0 upper=2.61 effort=200 velocity=30; type continuous -> revolute
- joint right_shoulder_pitch_joint: limit (none) -> lower=-2.87 upper=2.87 effort=100 velocity=30; type continuous -> revolute
- joint right_shoulder_roll_joint: limit (none) -> lower=-2.87 upper=2.87 effort=100 velocity=30; type continuous -> revolute
- joint right_shoulder_yaw_joint: limit (none) -> lower=-2.87 upper=2.87 effort=100 velocity=30; type continuous -> revolute

Commit message: 1

File: legged_gym/resources/robots/bhr8fc2/BHR8FC2.urdf (robot description, URDF)
Before this commit: robot BHR8FC2, 22 links, 21 joints
Links:
- link torso_link: mass 22.473048 -> 22.569164
Joints:
- joint left_ankle_pitch_joint: limit lower=-0.87 upper=0.52 effort=40 velocity=30 -> lower=-0.6108652381980153 upper=1.1344640137963142 effort=50 velocity=37
- joint left_ankle_roll_joint: limit lower=-0.35 upper=0.35 effort=40 velocity=30 -> lower=-0.3490658503988659 upper=0.3490658503988659 effort=50 velocity=37
- joint left_elbow_joint: limit lower=0.0 upper=2.61 effort=100 velocity=30 -> lower=0.17453292519943295 upper=2.007128639793479 effort=50 velocity=37
- joint left_hip_pitch_joint: limit lower=-1.92 upper=0.87 effort=200 velocity=30 -> lower=-0.4014257279586958 upper=1.6755160819145565 effort=88 velocity=32
- joint left_hip_roll_joint: limit lower=-0.52 upper=0.52 effort=150 velocity=30 -> lower=-0.5235987755982988 upper=0.5235987755982988 effort=88 velocity=32
- joint left_hip_yaw_joint: limit lower=-1.57 upper=1.57 effort=150 velocity=30 -> lower=-0.39269908169872414 upper=0.39269908169872414 effort=88 velocity=32
- joint left_knee_joint: limit lower=0.0 upper=2.61 effort=200 velocity=30 -> lower=0.20943951023931956 upper=2.2689280275926285 effort=139 velocity=20
- joint left_shoulder_pitch_joint: limit lower=-2.87 upper=2.87 effort=100 velocity=30 -> lower=-1.5707963267948966 upper=2.356194490192345 effort=88 velocity=32
- joint left_shoulder_roll_joint: limit lower=-2.87 upper=2.87 effort=100 velocity=30 -> lower=-0.17453292519943295 upper=1.5707963267948966 effort=88 velocity=32
- joint left_shoulder_yaw_joint: limit lower=-2.87 upper=2.87 effort=100 velocity=30 -> lower=-0.7853981633974483 upper=0.7853981633974483 effort=88 velocity=32
- joint right_ankle_pitch_joint: limit lower=-0.87 upper=0.52 effort=40 velocity=30 -> lower=-0.6108652381980153 upper=1.1344640137963142 effort=50 velocity=37
- joint right_ankle_roll_joint: limit lower=-0.35 upper=0.35 effort=40 velocity=30 -> lower=-0.3490658503988659 upper=0.3490658503988659 effort=50 velocity=37
- joint right_elbow_joint: limit lower=0.0 upper=2.61 effort=100 velocity=30 -> lower=0.17453292519943295 upper=2.007128639793479 effort=50 velocity=37
- joint right_hip_pitch_joint: limit lower=-1.92 upper=0.87 effort=200 velocity=30 -> lower=-0.4014257279586958 upper=1.6755160819145565 effort=88 velocity=32
- joint right_hip_roll_joint: limit lower=-0.52 upper=0.52 effort=150 velocity=30 -> lower=-0.5235987755982988 upper=0.5235987755982988 effort=88 velocity=32
- joint right_hip_yaw_joint: limit lower=-1.57 upper=1.57 effort=150 velocity=30 -> lower=-0.39269908169872414 upper=0.39269908169872414 effort=88 velocity=32
- joint right_knee_joint: limit lower=0.0 upper=2.61 effort=200 velocity=30 -> lower=0.20943951023931956 upper=2.2689280275926285 effort=139 velocity=20
- joint right_shoulder_pitch_joint: limit lower=-2.87 upper=2.87 effort=100 velocity=30 -> lower=-1.5707963267948966 upper=2.356194490192345 effort=88 velocity=32
- joint right_shoulder_roll_joint: limit lower=-2.87 upper=2.87 effort=100 velocity=30 -> lower=-0.17453292519943295 upper=1.5707963267948966 effort=88 velocity=32
- joint right_shoulder_yaw_joint: limit lower=-2.87 upper=2.87 effort=100 velocity=30 -> lower=-0.7853981633974483 upper=0.7853981633974483 effort=88 velocity=32

Commit message: 1

File: legged_gym/resources/robots/bhr8fc2/BHR8FC2.urdf (robot description, URDF)
Before this commit: robot BHR8FC2, 22 links, 21 joints
Joints:
- joint left_elbow_joint: limit lower=0.17453292519943295 upper=2.007128639793479 effort=50 velocity=37 -> lower=-2.007128639793479 upper=-0.17453292519943295 effort=50 velocity=37
- joint left_hip_yaw_joint: limit lower=-0.39269908169872414 upper=0.39269908169872414 effort=88 velocity=32 -> lower=-0.3490658503988659 upper=0.3490658503988659 effort=88 velocity=32
- joint left_knee_joint: limit lower=0.20943951023931956 upper=2.2689280275926285 effort=139 velocity=20 -> lower=-2.2689280275926285 upper=-0.20943951023931956 effort=139 velocity=20
- joint left_shoulder_pitch_joint: limit lower=-1.5707963267948966 upper=2.356194490192345 effort=88 velocity=32 -> lower=-2.356194490192345 upper=1.5707963267948966 effort=88 velocity=32
- joint left_shoulder_yaw_joint: limit lower=-0.7853981633974483 upper=0.7853981633974483 effort=88 velocity=32 -> lower=-0.7853981633974483 upper=1.5707963267948966 effort=88 velocity=32
- joint right_ankle_pitch_joint: limit lower=-0.6108652381980153 upper=1.1344640137963142 effort=50 velocity=37 -> lower=-1.1344640137963142 upper=0.6108652381980153 effort=50 velocity=37
- joint right_hip_pitch_joint: limit lower=-0.4014257279586958 upper=1.6755160819145565 effort=88 velocity=32 -> lower=-1.6755160819145565 upper=0.4014257279586958 effort=88 velocity=32
- joint right_hip_yaw_joint: limit lower=-0.39269908169872414 upper=0.39269908169872414 effort=88 velocity=32 -> lower=-0.3490658503988659 upper=0.3490658503988659 effort=88 velocity=32
- joint right_shoulder_roll_joint: limit lower=-0.17453292519943295 upper=1.5707963267948966 effort=88 velocity=32 -> lower=-1.5707963267948966 upper=0.17453292519943295 effort=88 velocity=32
- joint right_shoulder_yaw_joint: limit lower=-0.7853981633974483 upper=0.7853981633974483 effort=88 velocity=32 -> lower=-1.5707963267948966 upper=0.7853981633974483 effort=88 velocity=32

Commit message: 1

File: legged_gym/resources/robots/bhr8fc2/BHR8FC2.urdf (robot description, URDF)
Before this commit: robot BHR8FC2, 22 links, 21 joints
Joints:
- joint left_ankle_pitch_joint: limit lower=-0.6108652381980153 upper=1.1344640137963142 effort=50 velocity=37 -> lower=-0.6108652381980153 upper=1.1344640137963142 effort=145 velocity=32
- joint left_ankle_roll_joint: limit lower=-0.3490658503988659 upper=0.3490658503988659 effort=50 velocity=37 -> lower=-0.3490658503988659 upper=0.3490658503988659 effort=145 velocity=32
- joint left_elbow_joint: limit lower=-2.007128639793479 upper=-0.17453292519943295 effort=50 velocity=37 -> lower=-2.007128639793479 upper=-0.17453292519943295 effort=145 velocity=32
- joint left_hip_pitch_joint: limit lower=-0.4014257279586958 upper=1.6755160819145565 effort=88 velocity=32 -> lower=-0.4014257279586958 upper=1.6755160819145565 effort=145 velocity=32
- joint left_hip_roll_joint: limit lower=-0.5235987755982988 upper=0.5235987755982988 effort=88 velocity=32 -> lower=-0.5235987755982988 upper=0.5235987755982988 effort=145 velocity=32
- joint left_hip_yaw_joint: limit lower=-0.3490658503988659 upper=0.3490658503988659 effort=88 velocity=32 -> lower=-0.3490658503988659 upper=0.3490658503988659 effort=145 velocity=32
- joint left_knee_joint: limit lower=-2.2689280275926285 upper=-0.20943951023931956 effort=139 velocity=20 -> lower=-2.2689280275926285 upper=-0.20943951023931956 effort=145 velocity=32
- joint left_shoulder_pitch_joint: limit lower=-2.356194490192345 upper=1.5707963267948966 effort=88 velocity=32 -> lower=-2.356194490192345 upper=1.5707963267948966 effort=145 velocity=32
- joint left_shoulder_roll_joint: limit lower=-0.17453292519943295 upper=1.5707963267948966 effort=88 velocity=32 -> lower=-0.17453292519943295 upper=1.5707963267948966 effort=145 velocity=32
- joint left_shoulder_yaw_joint: limit lower=-0.7853981633974483 upper=1.5707963267948966 effort=88 velocity=32 -> lower=-0.7853981633974483 upper=1.5707963267948966 effort=145 velocity=32
- joint right_ankle_pitch_joint: limit lower=-1.1344640137963142 upper=0.6108652381980153 effort=50 velocity=37 -> lower=-1.1344640137963142 upper=0.6108652381980153 effort=145 velocity=32
- joint right_ankle_roll_joint: limit lower=-0.3490658503988659 upper=0.3490658503988659 effort=50 velocity=37 -> lower=-0.3490658503988659 upper=0.3490658503988659 effort=145 velocity=32
- joint right_elbow_joint: limit lower=0.17453292519943295 upper=2.007128639793479 effort=50 velocity=37 -> lower=0.17453292519943295 upper=2.007128639793479 effort=145 velocity=32
- joint right_hip_pitch_joint: limit lower=-1.6755160819145565 upper=0.4014257279586958 effort=88 velocity=32 -> lower=-1.6755160819145565 upper=0.4014257279586958 effort=145 velocity=32
- joint right_hip_roll_joint: limit lower=-0.5235987755982988 upper=0.5235987755982988 effort=88 velocity=32 -> lower=-0.5235987755982988 upper=0.5235987755982988 effort=145 velocity=32
- joint right_hip_yaw_joint: limit lower=-0.3490658503988659 upper=0.3490658503988659 effort=88 velocity=32 -> lower=-0.3490658503988659 upper=0.3490658503988659 effort=145 velocity=32
- joint right_knee_joint: limit lower=0.20943951023931956 upper=2.2689280275926285 effort=139 velocity=20 -> lower=0.20943951023931956 upper=2.2689280275926285 effort=145 velocity=32
- joint right_shoulder_pitch_joint: limit lower=-1.5707963267948966 upper=2.356194490192345 effort=88 velocity=32 -> lower=-1.5707963267948966 upper=2.356194490192345 effort=145 velocity=32
- joint right_shoulder_roll_joint: limit lower=-1.5707963267948966 upper=0.17453292519943295 effort=88 velocity=32 -> lower=-1.5707963267948966 upper=0.17453292519943295 effort=145 velocity=32
- joint right_shoulder_yaw_joint: limit lower=-1.5707963267948966 upper=0.7853981633974483 effort=88 velocity=32 -> lower=-1.5707963267948966 upper=0.7853981633974483 effort=145 velocity=32
