Commit message: 1

File: legged_gym/resources/robots/bhr8fc2/BHR8FC2.urdf (robot description, URDF)
Before this commit: robot BHR8FC2, 22 links, 21 joints
Joints:
- joint left_ankle_pitch_joint: limit lower=-0.6108652381980153 upper=1.1344640137963142 effort=145 velocity=32 -> lower=-0.6108652381980153 upper=1.1344640137963142 effort=120 velocity=20
- joint left_ankle_roll_joint: limit lower=-0.3490658503988659 upper=0.3490658503988659 effort=145 velocity=32 -> lower=-0.3490658503988659 upper=0.3490658503988659 effort=80 velocity=20
- joint left_elbow_joint: limit lower=-2.007128639793479 upper=-0.17453292519943295 effort=145 velocity=32 -> lower=-2.007128639793479 upper=-0.17453292519943295 effort=120 velocity=20
- joint left_hip_pitch_joint: limit lower=-0.4014257279586958 upper=1.6755160819145565 effort=145 velocity=32 -> lower=-0.4014257279586958 upper=1.6755160819145565 effort=120 velocity=20
- joint left_hip_roll_joint: limit lower=-0.5235987755982988 upper=0.5235987755982988 effort=145 velocity=32 -> lower=-0.5235987755982988 upper=0.5235987755982988 effort=120 velocity=20
- joint left_hip_yaw_joint: limit lower=-0.3490658503988659 upper=0.3490658503988659 effort=145 velocity=32 -> lower=-0.3490658503988659 upper=0.3490658503988659 effort=120 velocity=20
- joint left_knee_joint: limit lower=-2.2689280275926285 upper=-0.20943951023931956 effort=145 velocity=32 -> lower=-2.2689280275926285 upper=-0.20943951023931956 effort=150 velocity=20
- joint left_shoulder_pitch_joint: limit lower=-2.356194490192345 upper=1.5707963267948966 effort=145 velocity=32 -> lower=-2.356194490192345 upper=1.5707963267948966 effort=120 velocity=20
- joint left_shoulder_roll_joint: limit lower=-0.17453292519943295 upper=1.5707963267948966 effort=145 velocity=32 -> lower=-0.17453292519943295 upper=1.5707963267948966 effort=120 velocity=20
- joint left_shoulder_yaw_joint: limit lower=-0.7853981633974483 upper=1.5707963267948966 effort=145 velocity=32 -> lower=-0.7853981633974483 upper=1.5707963267948966 effort=120 velocity=20
- joint right_ankle_pitch_joint: limit lower=-1.1344640137963142 upper=0.6108652381980153 effort=145 velocity=32 -> lower=-1.1344640137963142 upper=0.6108652381980153 effort=120 velocity=20
- joint right_ankle_roll_joint: limit lower=-0.3490658503988659 upper=0.3490658503988659 effort=145 velocity=32 -> lower=-0.3490658503988659 upper=0.3490658503988659 effort=80 velocity=20
- joint right_elbow_joint: limit lower=0.17453292519943295 upper=2.007128639793479 effort=145 velocity=32 -> lower=0.17453292519943295 upper=2.007128639793479 effort=120 velocity=20
- joint right_hip_pitch_joint: limit lower=-1.6755160819145565 upper=0.4014257279586958 effort=145 velocity=32 -> lower=-1.6755160819145565 upper=0.4014257279586958 effort=120 velocity=20
- joint right_hip_roll_joint: limit lower=-0.5235987755982988 upper=0.5235987755982988 effort=145 velocity=32 -> lower=-0.5235987755982988 upper=0.5235987755982988 effort=120 velocity=20
- joint right_hip_yaw_joint: limit lower=-0.3490658503988659 upper=0.3490658503988659 effort=145 velocity=32 -> lower=-0.3490658503988659 upper=0.3490658503988659 effort=120 velocity=20
- joint right_knee_joint: limit lower=0.20943951023931956 upper=2.2689280275926285 effort=145 velocity=32 -> lower=0.20943951023931956 upper=2.2689280275926285 effort=150 velocity=20
- joint right_shoulder_pitch_joint: limit lower=-1.5707963267948966 upper=2.356194490192345 effort=145 velocity=32 -> lower=-1.5707963267948966 upper=2.356194490192345 effort=120 velocity=20
- joint right_shoulder_roll_joint: limit lower=-1.5707963267948966 upper=0.17453292519943295 effort=145 velocity=32 -> lower=-1.5707963267948966 upper=0.17453292519943295 effort=120 velocity=20
- joint right_shoulder_yaw_joint: limit lower=-1.5707963267948966 upper=0.7853981633974483 effort=145 velocity=32 -> lower=-1.5707963267948966 upper=0.7853981633974483 effort=120 velocity=20
